File: kicad/badge.kicad_sch (KiCad schematic)
At the start: 28 parts, among them U1 ATtiny85-20P, U2 4021, U3 74HC595, U4 74HC595

Commit message: Update badge with latest version
Signed-off-by: Josh Bressers <josh@bress.net>
Parts:
- added TP1, TP2, TP3, TP4, TP5, TP6, TP7, TP8: TestPoint, TestPoint:TestPoint_Pad_D1.0mm, symbol Connector:TestPoint
- R1, R10, R11, R12, R13, R14, R15, R16, R2, R3, R4, R5, R6, R7, R8, R9: footprint Resistor_THT:R_Axial_DIN0204_L3.6mm_D1.6mm_P7.62mm_Horizontal -> Resistor_THT:R_Axial_DIN0207_L6.3mm_D2.5mm_P10.16mm_Horizontal
Connections:
- net GND: now also TP4.1
- net VCC: now also TP8.1
- net at R13.1, U2.4 (D3): now also S4.4; no longer S4.3
- net at R11.1, U2.14 (D5): now also S6.4; no longer S6.3
- net at R14.1, U2.5 (D2): now also S3.4; no longer S3.3
- net at R15.1, U2.6 (D1): now also S2.4; no longer S2.3
- net at R16.1, U2.7 (D0): now also S1.4; no longer S1.3
- net at U1.7 (PB2), U2.10 (CP), U3.11 (SRCLK)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: now also TP7.1
- net at R12.1, U2.13 (D4): now also S5.4; no longer S5.3
- net at U1.3 (XTAL2/PB4), U2.3 (Q7): now also TP3.1
- net at U1.6 (PB1), U2.9 (PL), U3.12 (RCLK)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: now also TP6.1
- net at U1.2 (XTAL1/PB3), U3.14 (SER): now also TP2.1
- net at U1.1 (~{RESET}/PB5): now also TP1.1
- net at U1.5 (AREF/PB0), U4.14 (SER): now also TP5.1

Commit message: Update badge PCB
Signed-off-by: Josh Bressers <josh@bress.net>
Parts:
- TP1, TP2, TP3, TP4, TP5, TP6, TP7, TP8: footprint TestPoint:TestPoint_Pad_D1.0mm -> TestPoint:TestPoint_THTPad_D1.5mm_Drill0.7mm
Changed lines of the file:
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@@
       (effects (font (size 1.27 1.27)) (justify left) hide)
     )
-    (property "Footprint" "TestPoint:TestPoint_Pad_D1.0mm" (at 143.51 54.61 0)
+    (property "Footprint" "TestPoint:TestPoint_THTPad_D1.5mm_Drill0.7mm" (at 143.51 54.61 0)
       (effects (font (size 1.27 1.27)) hide)
     )
@@
       (effects (font (size 1.27 1.27)) (justify left) hide)
     )
-    (property "Footprint" "TestPoint:TestPoint_Pad_D1.0mm" (at 143.51 57.15 0)
+    (property "Footprint" "TestPoint:TestPoint_THTPad_D1.5mm_Drill0.7mm" (at 143.51 57.15 0)
       (effects (font (size 1.27 1.27)) hide)
     )
@@
       (effects (font (size 1.27 1.27)) (justify left) hide)
     )
-    (property "Footprint" "TestPoint:TestPoint_Pad_D1.0mm" (at 143.51 46.99 0)
+    (property "Footprint" "TestPoint:TestPoint_THTPad_D1.5mm_Drill0.7mm" (at 143.51 46.99 0)
       (effects (font (size 1.27 1.27)) hide)
     )
@@
       (effects (font (size 1.27 1.27)) (justify left) hide)
     )
-    (property "Footprint" "TestPoint:TestPoint_Pad_D1.0mm" (at 143.51 39.37 0)
+    (property "Footprint" "TestPoint:TestPoint_THTPad_D1.5mm_Drill0.7mm" (at 143.51 39.37 0)
       (effects (font (size 1.27 1.27)) hide)
     )
@@
       (effects (font (size 1.27 1.27)) (justify left) hide)
     )
-    (property "Footprint" "TestPoint:TestPoint_Pad_D1.0mm" (at 143.51 49.53 0)
+    (property "Footprint" "TestPoint:TestPoint_THTPad_D1.5mm_Drill0.7mm" (at 143.51 49.53 0)
       (effects (font (size 1.27 1.27)) hide)
     )
@@
       (effects (font (size 1.27 1.27)) (justify left) hide)
     )
-    (property "Footprint" "TestPoint:TestPoint_Pad_D1.0mm" (at 143.51 52.07 0)
+    (property "Footprint" "TestPoint:TestPoint_THTPad_D1.5mm_Drill0.7mm" (at 143.51 52.07 0)
       (effects (font (size 1.27 1.27)) hide)
     )
@@
       (effects (font (size 1.27 1.27)) (justify left) hide)
     )
-    (property "Footprint" "TestPoint:TestPoint_Pad_D1.0mm" (at 143.51 44.45 0)
+    (property "Footprint" "TestPoint:TestPoint_THTPad_D1.5mm_Drill0.7mm" (at 143.51 44.45 0)
       (effects (font (size 1.27 1.27)) hide)
     )
@@
       (effects (font (size 1.27 1.27)) (justify left) hide)
     )
-    (property "Footprint" "TestPoint:TestPoint_Pad_D1.0mm" (at 143.51 41.91 0)
-      (effects (font (size 1.27 1.27)) hide)
-    )
+    (property "Footprint" "TestPoint:TestPoint_THTPad_D1.5mm_Drill0.7mm" (at 143.51 41.91 0)
+      (effects (font (size 1.27 1.27)) hide)
+    )
